File: KiCad/OM-FlexGrid V1/OM-FlexGrid-Rigid-PCB/OM-FlexGrid-Rigid-PCB.kicad_pcb (KiCad board)
At the start: 4 copper layers, 31.6 x 56.1 mm, 47 parts, among them IC1 ICM-42688-P, J1 Conn_01x08_Pin, J2 BAT Terminal, J3 Conn_01x21_Pin, J4 USB_C_Receptacle, J5 Conn_01x02, Q1 IRLML2060, Q2 VP0610T, Q3 IRLML2060, U1 CD74HC4067M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

Commit message: FlexGrid V1
Parts:
- removed R16: 10k, Resistor_SMD:R_0603_1608Metric
- added H1: MountingHole_Pad, MountingHole:MountingHole_2.2mm_M2, F.Cu at (157.0, 103.5)
- added H2: MountingHole_Pad, MountingHole:MountingHole_2.2mm_M2, F.Cu at (212.0, 104.0)
- added H3: MountingHole_Pad, MountingHole:MountingHole_2.2mm_M2, F.Cu at (212.0, 126.0)
- added H4: MountingHole_Pad, MountingHole:MountingHole_2.2mm_M2, F.Cu at (157.0, 126.5)
- added J6: Conn_01x03_Pin, Connector_PinHeader_1.27mm:PinHeader_1x03_P1.27mm_Vertical, F.Cu at (162.2, 121.8)
- J1: value Conn_01x08_Pin -> Conn_01x06_Pin; footprint Connector_PinHeader_2.54mm:PinHeader_1x08_P2.54mm_Vertical -> Connector_PinHeader_1.27mm:PinHeader_2x03_P1.27mm_Vertical
- J3: value Conn_01x21_Pin -> Conn_01x19_Pin; footprint Connector_PinSocket_2.54mm:PinSocket_1x21_P2.54mm_Vertical -> Connector_PinHeader_1.27mm:PinHeader_1x19_P1.27mm_Vertical
- moved J2 87.8 mm to (215.5, 115.5)
- moved J5 84.5 mm to (214.5, 108.0), turned to 90 degrees
- moved R10 81.2 mm to (210.2, 120.5), turned to 0 degrees
- moved C9 80.6 mm to (213.0, 120.3)
- moved D4 79.6 mm to (213.3, 111.0), turned to 180 degrees
- moved Q1 76.3 mm to (210.1, 114.6), turned to 90 degrees
- moved J3 75.3 mm to (195.9, 127.0), turned to -90 degrees
- moved R11 74.7 mm to (210.2, 118.0), turned to 0 degrees
- moved SCRN1 69.8 mm to (188.3, 124.0), turned to -90 degrees
- moved D2 67.0 mm to (185.1, 104.2)
- moved R5 66.7 mm to (185.4, 100.5)
- moved BOOT1 66.1 mm to (206.2, 103.4)
- moved C10 66.1 mm to (207.2, 112.5)
- moved C5 66.1 mm to (207.2, 109.5)
- moved C8 66.1 mm to (184.2, 108.5)
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Connections:
- net GP33 renamed GP40
- J1 pad 1: GND -> GP41
- J1 pad 2: +3V3 -> SPI_MOSI
- J1 pad 4: SPI_MOSI -> SPI_MISO
- J1 pad 5: SPI_MISO -> CS
- J3 pad 1: GND -> COL_0
- J3 pad 10: COL_7 -> COL_9
- J3 pad 11: COL_8 -> COL_10
- J3 pad 12: COL_9 -> COL_11
- J3 pad 13: COL_10 -> COL_12
- J3 pad 14: COL_11 -> COL_13
- J3 pad 15: COL_12 -> COL_14
- J3 pad 16: COL_13 -> ROW_0
- J3 pad 17: COL_14 -> ROW_1
- J3 pad 18: ROW_0 -> ROW_2
- J3 pad 19: ROW_1 -> ROW_3
- J3 pad 2: +3V3 -> COL_1
- J3 pad 3: COL_0 -> COL_2
- J3 pad 4: COL_1 -> COL_3
- J3 pad 5: COL_2 -> COL_4
- J3 pad 6: COL_3 -> COL_5
- J3 pad 7: COL_4 -> COL_6
- J3 pad 8: COL_5 -> COL_7
- J3 pad 9: COL_6 -> COL_8
- U2 pad 34: GP34 -> GP41
Routing:
- net ROW_3: track 3.20 -> 71.8 mm, vias 0 -> 3
- net GP40: track 0.00 -> 57.7 mm, vias 0 -> 1
- net ROW_1: track 2.91 -> 59.6 mm, vias 0 -> 1
- net MOT_SIG: track 0.00 -> 51.7 mm
- net GP41: track 0.00 -> 48.4 mm, vias 0 -> 1
- net VBAT: track 35.3 -> 83.2 mm
- net 100: track 0.00 -> 47.6 mm, vias 0 -> 1
- net ROW_0: track 3.14 -> 47.9 mm, vias 0 -> 1
- net S1: track 0.00 -> 33.2 mm, vias 0 -> 2
- net COL_14: track 0.00 -> 32.6 mm
- net S0: track 0.00 -> 32.4 mm, vias 0 -> 2
- net D-: track 2.99 -> 34.6 mm, vias 0 -> 1
- net COL_13: track 0.00 -> 30.4 mm
- net EN: track 11.6 -> 41.8 mm, vias 0 -> 1
- net D+: track 2.99 -> 32.5 mm, vias 0 -> 1
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Other:
- board size 31.6 x 56.1 mm -> 65.5 x 33 mm

Commit message: V1-1
Parts:
- added C12: 2.2 uF, Capacitor_SMD:C_0603_1608Metric, F.Cu at (172.9, 136.2)
- added C13: 2.2 uF, Capacitor_SMD:C_0603_1608Metric, F.Cu at (172.9, 134.2)
- added C14: 2.2 uF, Capacitor_SMD:C_0603_1608Metric, F.Cu at (172.9, 131.8)
- added C15: 2.2 uF, Capacitor_SMD:C_0603_1608Metric, F.Cu at (172.9, 129.4)
- added J7: Conn_01x02_Pin, Connector_PinSocket_2.00mm:PinSocket_1x02_P2.00mm_Vertical, F.Cu at (178.3, 143.7)
- moved H4 44.1 mm to (172.7, 85.2), turned to -90 degrees
- moved SELECT1 43.0 mm to (183.8, 85.1), turned to 0 degrees
- moved H1 42.7 mm to (195.7, 85.2), turned to -90 degrees
- moved J2 42.6 mm to (183.7, 143.8), turned to 90 degrees
- moved MENU1 42.3 mm to (189.9, 85.1), turned to 0 degrees
- moved J5 41.9 mm to (191.2, 142.8), turned to 0 degrees
- moved H3 41.4 mm to (173.2, 140.2), turned to -90 degrees
- moved R15 40.1 mm to (172.0, 88.8), turned to 180 degrees
- moved C9 40.1 mm to (178.9, 141.2), turned to 0 degrees
- moved H2 40.0 mm to (195.2, 140.2), turned to -90 degrees
- moved D4 39.6 mm to (188.2, 141.6), turned to 90 degrees
- moved R10 36.3 mm to (178.7, 138.4), turned to -90 degrees
- moved R14 36.2 mm to (172.0, 92.0), turned to 180 degrees
- moved R11 35.5 mm to (181.2, 138.4), turned to -90 degrees
- moved J3 35.1 mm to (172.2, 101.2), turned to 0 degrees
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Routing:
- net ROW_3: track 71.8 -> 132.1 mm
- net ROW_2: track 30.6 -> 84.9 mm
- net ROW_1: track 59.6 -> 103.0 mm
- net ROW_0: track 47.9 -> 80.2 mm
- net COL_8: track 17.6 -> 34.6 mm
- net COL_0: track 15.3 -> 28.9 mm
- net COL_9: track 21.1 -> 32.6 mm
- net COL_1: track 15.5 -> 25.5 mm
- net COL_2: track 15.5 -> 25.4 mm
- net COL_14: track 32.6 -> 22.9 mm
- net COL_3: track 15.8 -> 24.8 mm
- net COL_4: track 16.0 -> 23.9 mm
- net S1: track 33.2 -> 25.7 mm
- net COL_10: track 23.5 -> 30.7 mm
- net GND: track 75.9 -> 82.8 mm, vias 21 -> 24
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Other:
- board size 65.5 x 33 mm -> 33 x 65.5 mm
