File: KiCad/OM-FlexGrid V1/OM-FlexGrid-Rigid-PCB/OM-FlexGrid-Rigid-PCB.kicad_sch (KiCad schematic)
At the start: 47 parts, among them IC1 ICM-42688-P, J1 Conn_01x08_Pin, J2 BAT Terminal, J3 Conn_01x21_Pin, J4 USB_C_Receptacle, J5 Conn_01x02, Q1 IRLML2060, Q2 VP0610T, Q3 IRLML2060, U1 CD74HC4067M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

Commit message: FlexGrid V1
Parts:
- removed J1: Conn_01x08_Pin, Connector_PinHeader_2.54mm:PinHeader_1x08_P2.54mm_Vertical, symbol Connector:Conn_01x08_Pin
- removed J3: Conn_01x21_Pin, Connector_PinSocket_2.54mm:PinSocket_1x21_P2.54mm_Vertical, symbol Connector:Conn_01x21_Pin
- removed R16: 10k, Resistor_SMD:R_0603_1608Metric, symbol Device:R
- added H1, H2, H3, H4: MountingHole_Pad, MountingHole:MountingHole_2.2mm_M2, symbol Mechanical:MountingHole_Pad
- added J1: Conn_01x06_Pin, Connector_PinHeader_1.27mm:PinHeader_2x03_P1.27mm_Vertical, symbol Connector:Conn_01x06_Pin
- added J3: Conn_01x19_Pin, Connector_PinHeader_1.27mm:PinHeader_1x19_P1.27mm_Vertical, symbol Connector:Conn_01x19_Pin
- added J6: Conn_01x03_Pin, Connector_PinHeader_1.27mm:PinHeader_1x03_P1.27mm_Vertical, symbol Connector:Conn_01x03_Pin
Connections:
- net COL_0: now also J3.1 (Pin_1)
- net COL_1: now also J3.2 (Pin_2)
- net COL_10: now also J3.11 (Pin_11)
- net COL_11: now also J3.12 (Pin_12)
- net COL_12: now also J3.13 (Pin_13)
- net COL_13: now also J3.14 (Pin_14)
- net COL_14: now also J3.15 (Pin_15)
- net COL_2: now also J3.3 (Pin_3)
- net COL_3: now also J3.4 (Pin_4)
- net COL_4: now also J3.5 (Pin_5)
- net COL_5: now also J3.6 (Pin_6)
- net COL_6: now also J3.7 (Pin_7)
- net COL_7: now also J3.8 (Pin_8)
- net COL_8: now also J3.9 (Pin_9)
- net COL_9: now also J3.10 (Pin_10)
- net CS: now also J1.5 (Pin_5)
- net GND: now also J6.1 (Pin_1)
- net ROW_0: now also J3.16 (Pin_16)
- net ROW_1: now also J3.17 (Pin_17)
- net ROW_2: now also J3.18 (Pin_18)
- net ROW_3: now also J3.19 (Pin_19)
- net RX: now also J6.2 (Pin_2)
- net SPI_MISO: now also J1.4 (Pin_4)
- net SPI_MOSI: now also J1.2 (Pin_2)
- net SPI_SCK: now also J1.3 (Pin_3)
- net TX: now also J6.3 (Pin_3)
- net GP33 renamed GP40
- net GP40: now also J1.6 (Pin_6)
- net GP34 renamed GP41
- net GP41: now also J1.1 (Pin_1)
Other:
- moved on the sheet: R12, R13, R14, R15, U1

Commit message: V1-1
Parts:
- added C12, C13, C14, C15: 2.2 uF, Capacitor_SMD:C_0603_1608Metric, symbol Device:C
- added J7: Conn_01x02_Pin, Connector_PinSocket_2.00mm:PinSocket_1x02_P2.00mm_Vertical, symbol Connector:Conn_01x02_Pin
Connections:
- net +3V3: now also J7.2 (Pin_2)
- net GND: now also C12.1, C13.1, C14.1, C15.1, J7.1 (Pin_1)
- net ROW_0: now also C12.2
- net ROW_1: now also C13.2
- net ROW_2: now also C14.2
- net ROW_3: now also C15.2
Other:
- moved on the sheet: J3, R12, R13, R14, R15
