File: KiCad/OM-FlexGrid V2/OM-FlexGrid-Rigid-PCB/OM-FlexGrid-Rigid-PCB.kicad_sch (KiCad schematic)
At the start: 56 parts, among them IC1 ICM-42688-P, J1 Conn_01x06_Pin, J2 BAT Terminal, J3 Conn_01x19_Pin, J4 USB_C_Receptacle, J5 Conn_01x02, J6 Conn_01x03_Pin, J7 Conn_01x02_Pin, Q1 IRLML2060, Q2 VP0610T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

Commit message: Cleanup V2-1
Parts:
- Q2: value VP0610T -> VP0610T or BSS84
- U4: value LTC4054ES5-4.2 -> LTC4054ES5-4.2 or STC4054GR
Changed lines of the file:
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@@
 		(on_board yes)
 		(dnp no)
-		(fields_autoplaced yes)
 		(property "Reference" "Q2"
 			(at 26.67 92.71 90)
@@
 			)
 		)
-		(property "Value" "VP0610T"
-			(at 26.67 95.25 90)
+		(property "Value" "VP0610T or BSS84"
+			(at 30.48 95.25 90)
 			(effects
 				(font
@@
 			)
 		)
-		(property "Value" "LTC4054ES5-4.2"
-			(at 129.54 99.06 0)
-			(effects
-				(font
+		(property "Value" "LTC4054ES5-4.2 or STC4054GR"
+			(at 125.984 99.06 0)
+			(effects
+				(font
