File: KiCad/OM-FlexGrid V3/OM-FlexGrid-Rigid-PCB/OM-FlexGrid-Rigid-PCB.kicad_sch (KiCad schematic)
At the start: 56 parts, among them IC1 ICM-42688-P, J1 Conn_01x06_Pin, J2 BAT Terminal, J3 Conn_01x20, J4 USB_C_Receptacle, J5 Conn_01x02, J6 Conn_01x03_Pin, J7 Conn_01x02_Pin, Q1 IRLML2060, Q2 VP0610T or BSS84, Q3 IRLML2060, U1 CD74HC4067M, U2 ESP32-S3-WROOM-1-N16R8, U3 TPS7A03, U4 LTC4054ES5-4.2 or STC4054GR

Commit message: V3 Rigid PCB: align schematic with BOM and exclude hand-soldered parts from JLC fab
- Fix D1 footprint label: 1N4007 -> 1N5819 (Schottky, matches BOM)
- Fix C9 value: 100 uF -> 22 uF (matches BOM)
- Normalize cap notation 0.1 uF -> 100 nF
- List ICM-42688-P / ICM-42670-L alternatives on IC1
- Mark connectors (J1-J7), switches (BOOT1, SW_PWR1, SW_RST1, SELECT1, MENU1)
  and screen (SCRN1) as exclude_from_pos_files + exclude_from_bom so JLC SMT
  assembly does not try to place them

Co-Authored-By: Claude Opus 4.7 <noreply@anthropic.com>
Parts:
- C10: value 0.1 uF -> 100 nF
- C9: value 100 uF -> 22 uF
- D4: value 1N4007 -> 1N5819
- IC1: value ICM-42688-P -> ICM-42688-P or ICM-42670-L
Changed lines of the file:
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@@
 			)
 		)
-		(property "Value" "0.1 uF"
+		(property "Value" "100 nF"
 			(at 259.08 154.9399 0)
 			(effects
@@
 			)
 		)
-		(property "Value" "1N4007"
+		(property "Value" "1N5819"
 			(at 34.29 162.56 90)
 			(effects
@@
 			)
 		)
-		(property "Value" "ICM-42688-P"
+		(property "Value" "ICM-42688-P or ICM-42670-L"
 			(at 239.522 130.048 0)
 			(effects
@@
 			)
 		)
-		(property "Value" "100 uF"
+		(property "Value" "22 uF"
 			(at 47.371 162.433 0)
 			(effects
