File: KiCad/OM-FlexGrid V3/OM-FlexGrid-Rigid-PCB/OM-FlexGrid-Rigid-PCB.kicad_sch (KiCad schematic)
At the start: 56 parts, among them IC1 ICM-42688-P, J1 Conn_01x06_Pin, J2 BAT Terminal, J3 Conn_01x20, J4 USB_C_Receptacle, J5 Conn_01x02, J6 Conn_01x03_Pin, J7 Conn_01x02_Pin, Q1 IRLML2060, Q2 VP0610T or BSS84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

Commit message: V3 release - 20-pin FFC interconnect (ordered, untested)
- Switch flex-to-rigid interconnect to Wurth 687120183722 ZIF FFC
- Integrated stiffened FFC tail on flex (FR4, 0.20 mm, bottom side)
- Widen FFC tail to 11.1 mm to meet Wurth 0.8 mm side margin spec
- Add V3 gerber bundles (flex + rigid), rigid BOM CSV, V3 schematic PDF
- Update top-level README to highlight V3 as latest revision
- Rename schematic PDFs: Rigit -> Rigid
- Clean up legacy V1/V2 gerber duplicates from V3 folder
Other:
- company: (none) -> Open Muscle
- title: (none) -> Open Muscle FlexGrid Rigid PCB V3
Changed lines of the file:
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@@
 	(generator_version "9.0")
 	(paper "A4")
+	(title_block
+		(title "Open Muscle FlexGrid Rigid PCB V3")
+		(rev "V3")
+		(company "Open Muscle")
+	)
 	(rectangle
 		(start 13.97 85.09)
