File: KiCad/OM-FlexGrid V3/OM-FlexGrid-Flex/OM-FlexGrid-Flex.kicad_pcb (KiCad board)
At the start: 2 copper layers, 260 x 109.7 mm, 61 parts, among them J1 Conn_01x20

Commit message: V3 release - 20-pin FFC interconnect (ordered, untested)
- Switch flex-to-rigid interconnect to Wurth 687120183722 ZIF FFC
- Integrated stiffened FFC tail on flex (FR4, 0.20 mm, bottom side)
- Widen FFC tail to 11.1 mm to meet Wurth 0.8 mm side margin spec
- Add V3 gerber bundles (flex + rigid), rigid BOM CSV, V3 schematic PDF
- Update top-level README to highlight V3 as latest revision
- Rename schematic PDFs: Rigit -> Rigid
- Clean up legacy V1/V2 gerber duplicates from V3 folder
Other:
- board size 260 x 109.7 mm -> 260 x 109.6 mm

Commit message: Add FlexGrid V4 design with onboard SD card; clean up backups
V4 rigid and flex PCB design. Adds an onboard microSD card so the band can log capture sessions standalone, without a tethered PC. V4 3D and animation assets (Blender, glTF, STEP) are tracked via Git LFS.

Also stop versioning KiCad and Blender auto-backups (*-backups/, *.blend[0-9]) and remove the old backup archives.

Suggested-by: Kyle.T.Y <64039282+HeatRIderHR@users.noreply.github.com>
Routing:
- net COL_14: track 64.6 -> 70.1 mm
- net ROW_3: track 99.7 -> 102.6 mm
Other:
- outline, holes or cut-outs redrawn
