File: KiCad/OM-FlexGrid V4/OM-FlexGrid-Rigid-PCB/OM-FlexGrid-Rigid-PCB.kicad_pcb (KiCad board)
At the start: 4 copper layers, 33 x 65.5 mm, 62 parts, among them IC1 ICM-42688-P, J1 Conn_01x06_Pin, J2 BAT Terminal, J3 Conn_01x20, J4 USB_C_Receptacle, J5 Conn_01x02, J6 Conn_01x03_Pin, J7 Conn_01x02_Pin, J9 Micro_SD_Card, Q1 IRLML2060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

Commit message: V4 Rigid PCB: fix USBLC6 pinout + expand JLC-assembled BOM
USBLC6 ESD chip fix
-------------------
Swap the VBUS and GND power-flag connections on the USBLC6-2SC6
footprint in the schematic. Earlier revision wired pin 2 to VBUS
and pin 5 to GND, but the actual chip pinout is pin 2 = GND and
pin 5 = VCC. Result on the first populated V4 board was that the
USB enumerated VBUS (Windows chime) but the data lines were
clamped to garbage by the now-forward-biased internal ESD diodes,
so no COM port was assigned and esptool could not sync.

Workaround on the first board was to rotate the USBLC6 180 degrees
during placement (SOT-23-6 footprint is symmetric, so the I/O pin
pairs route correctly either way; only VCC/GND end up reversed).
This commit puts the corrected pinout into the schematic so the
next fab order from anyone (including community members pulling
from GitHub) gets a board that works without manual rework.

PCB regenerated against the new schematic. All gerbers, drill
files, BOM, and CPL are refreshed accordingly. GERBER zip in
jlcpcb/production_files/ is the as-ready-to-upload archive.

BOM expansion
-------------
While re-running the JLCPCB plugin, additional designators were
toggled to BOM-ON for JLC assembly (previously hand-solder):
  - C9 (100uF cap)
  - R10, R11 (10k pulldowns)
  - Q1 (IRLML2060)
  - J1 (programming header)
  - J7 (pin socket)
That reduces the hand-solder workload from earlier V4 plan; the
remaining hand-solder items are still the ESP32 module, mux,
microSD socket, USB-C, and Wurth FFC connector. Update the
README hand-solder list before the next bring-up if these counts
matter to anyone following along.

3D models
---------
Adds WRL export and an updated Blender file for the V4 board
revision so the mechanical fit-check renders match the corrected
layout. FlexGridV5.blend has been touched alongside as well
(no V4 functional implication).

Production output folder
------------------------
Adds a parallel production/ folder generated by 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
Parts:
- turned U5 to 180 degrees
Connections:
- U5 pad 1: D+ -> Net-(J4-D--PadA7)
- U5 pad 2: VBUS -> GND
- U5 pad 3: D- -> Net-(J4-D+-PadA6)
- U5 pad 4: Net-(J4-D--PadA7) -> D+
- U5 pad 5: GND -> VBUS
- U5 pad 6: Net-(J4-D+-PadA6) -> D-
Routing:
- net GND: vias 34 -> 35
